File: labs/6-pcb/pcb_lab_v2_base/pcb_lab_v2_base.kicad_pcb (KiCad board)
At the start: 2 copper layers, 64.5 x 25 mm, 8 parts, among them J1 Raspberry_Pi_2_3, J2 UART

Commit message: minor
Connections:
- J1 pad 1: +3V3 -> unconnected-(J1-3V3-Pad1)_1
- J1 pad 17: +3V3 -> unconnected-(J1-3V3-Pad1)
Routing:
- net Net-(D2-DOUT): track 0.00 -> 7.45 mm
- net Net-(D1-DOUT): track 0.00 -> 7.45 mm
Other:
- board text added: "JLCJLCJLCJLC"
