File: labs/6-pcb/pcb_lab_v2_base/pcb_lab_v2_base.kicad_sch (KiCad schematic)
At the start: 8 parts, among them J1 Raspberry_Pi_2_3, J2 UART

Commit message: minor
Connections:
- net +3V3: no longer names the net of J1.1 (3V3), J1.17 (3V3)
- no-connect marks 27 -> 28
